File: hermod-extended/left/hermod.kicad_pcb (KiCad board)
At the start: 2 copper layers, 189.2 x 139.5 mm, 187 parts, among them J1 USB_C_Receptacle_USB2.0, J2 Conn_01x05, J3 USB_C_Receptacle_USB2.0, Q1 AO3401A, Q2 MMUN2233LT1G, U1 STM32F072CBT6, U2 PRTR5V0U2X, U3 XC6206PxxxMR-Regulator_Linear, U4 CR2013-MI2120, U5 TXB0101

Commit message: Finished routing the left side 100%
Parts:
- removed R5: 0, Resistor_SMD:R_0402_1005Metric
Routing:
- net D+: track 23.2 -> 24.6 mm
