File: mist/matrix.kicad_sch (KiCad schematic)
At the start: 206 parts

Commit message: Update og mist, updated readmes
Parts:
- added S1, S3: MX_stab, PCM_marbastlib-mx:STAB_MX_P_2.25u, symbol PCM_marbastlib-mx:MX_stab
- added S2: MX_stab, PCM_marbastlib-mx:STAB_MX_P_2.75u, symbol PCM_marbastlib-mx:MX_stab
- added S4, S5, S6, S7: MX_stab, PCM_marbastlib-mx:STAB_MX_P_2u, symbol PCM_marbastlib-mx:MX_stab
