File: mist-udb-mk-ii-north/mist.kicad_sch (KiCad schematic)
At the start: 32 parts, among them J1 78171-0004, J2 Conn_01x05, Q3 MMUN2133LT1G, U3 XC6206PxxxMR-Regulator_Linear, U4 CR2013-MI2120, U5 STM32G474RETx, U6 SN74AHCT1G125DBVR

Commit message: Fixed cap annotations
Parts:
- renumbered D40 to D110, D41 to D111
Changed lines of the file:
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@@
 (kicad_sch
-	(version 20231120)
+	(version 20250114)
 	(generator "eeschema")
-	(generator_version "8.0")
+	(generator_version "9.0")
 	(paper "A3")
+	(text "Decoupling Capacitors"
+		(exclude_from_sim no)
+		(at 118.745 145.415 0)
+		(effects
+			(font
+				(size 1.27 1.27)
+			)
+			(justify left bottom)
+		)
+	)
+	(text "NOTE:\n  BOOT0: L=0.99V, H=2.31V\n    nRST: L=0.99V, H=2.31V\nRC network value designed to ensure\nthat at time of sampling:\nnRST=2.31V=H, BOOT0=2.75V=H"
+		(exclude_from_sim no)
+		(at 288.036 175.768 0)
+		(effects
+			(font
+				(size 1.27 1.27)
+			)
+			(justify left bottom)
+		)
+	)
+	(text "Power Regulation"
+		(exclude_from_sim no)
+		(at 207.01 59.055 0)
+		(effects
+			(font
+				(size 1.27 1.27)
+			)
+			(justify left bottom)
+		)
+	)
+	(text "Reset Circuit"
+		(exclude_from_sim no)
+		(at 250.698 149.606 0)
+		(effects
+			(font
+				(size 2.54 2.54)
+				(thickness 0.508)
+				(bold yes)
+				(italic yes)
+			)
+			(justify left bottom)
+		)
+	)
+	(text "Software Debug"
+		(exclude_from_sim no)
+		(at 199.644 110.49 0)
+		(effects
+			(font
+				(size 1.27 1.27)
+			)
+			(justify left bottom)
+		)
+	)
+	(text "NRST has internal pull-up.\nCapacitor holds signal stable.\nOptionally, remove the button,\nand reset by power-cycling the board."
+		(exclude_from_sim no)
+		(at 200.66 104.14 0)
+		(effects
+			(font
+				(size 1.27 1.27)
+			)
+			(justify left bottom)
+		)
+	)
+	(text "Level Shifter\nTo convert the 3.3v signal to 5v\nfor the SK6812 LEDs."
+		(exclude_from_sim no)
+		(at 256.032 77.978 0)
+		(effects
+			(font
+				(size 1.27 1.27)
+			)
+			(justify left bottom)
+		)
+	)
+	(text "LCD Display"
+		(exclude_from_sim no)
+		(at 136.906 88.138 0)
+		(effects
+			(font
+				(size 2.54 2.54)
+				(thickness 0.508)
+				(bold yes)
+				(italic yes)
+			)
+			(justify left bottom)
+		)
+	)
 	(junction
 		(at 262.89 175.26)
@@
 		)
 	)
-	(text "Decoupling Capacitors"
-		(exclude_from_sim no)
-		(at 118.745 145.415 0)
-		(effects
-			(font
-				(size 1.27 1.27)
-			)
-			(justify left bottom)
-		)
-	)
-	(text "NOTE:\n  BOOT0: L=0.99V, H=2.31V\n    nRST: L=0.99V, H=2.31V\nRC network value designed to ensure\nthat at time of sampling:\nnRST=2.31V=H, BOOT0=2.75V=H"
-		(exclude_from_sim no)
-		(at 288.036 175.768 0)
-		(effects
-			(font
-				(size 1.27 1.27)
-			)
-			(justify left bottom)
-		)
-	)
-	(text "Power Regulation"
-		(exclude_from_sim no)
-		(at 207.01 59.055 0)
-		(effects
-			(font
-				(size 1.27 1.27)
-			)
-			(justify left bottom)
-		)
-	)
-	(text "Reset Circuit"
-		(exclude_from_sim no)
-		(at 250.698 149.606 0)
-		(effects
-			(font
-				(size 2.54 2.54)
-				(thickness 0.508)
-				(bold yes)
-				(italic yes)
-			)
-			(justify left bottom)
-		)
-	)
-	(text "Software Debug"
-		(exclude_from_sim no)
-		(at 199.644 110.49 0)
-		(effects
-			(font
-				(size 1.27 1.27)
-			)
-			(justify left bottom)
-		)
-	)
-	(text "NRST has internal pull-up.\nCapacitor holds signal stable.\nOptionally, remove the button,\nand reset by power-cycling the board."
-		(exclude_from_sim no)
-		(at 200.66 104.14 0)
-		(effects
-			(font
-				(size 1.27 1.27)
-			)
-			(justify left bottom)
-		)
-	)
-	(text "Level Shifter\nTo convert the 3.3v signal to 5v\nfor the SK6812 LEDs."
-		(exclude_from_sim no)
-		(at 256.032 77.978 0)
-		(effects
-			(font
-				(size 1.27 1.27)
-			)
-			(justify left bottom)
-		)
-	)
-	(text "LCD Display"
-		(exclude_from_sim no)
-		(at 136.906 88.138 0)
-		(effects
-			(font
-				(size 2.54 2.54)
-				(thickness 0.508)
-				(bold yes)
-				(italic yes)
-			)
-			(justify left bottom)
-		)
-	)
 	(global_label "col8"
 		(shape input)
@@
 		(on_board yes)
 		(dnp no)
-		(property "Reference" "D41"
+		(property "Reference" "D111"
 			(at 224.282 173.8884 90)
 			(effects
@@
 			(project "hermod-left"
 				(path "/cb32b2da-a60d-4ed4-a57b-2c397f553171"
-					(reference "D41")
+					(reference "D111")
 					(unit 1)
 				)
@@
 		(on_board yes)
 		(dnp no)
-		(property "Reference" "D40"
+		(property "Reference" "D110"
 			(at 224.282 158.8516 90)
 			(effects
@@
 			(project "hermod-left"
 				(path "/cb32b2da-a60d-4ed4-a57b-2c397f553171"
-					(reference "D40")
+					(reference "D110")
 					(unit 1)
 				)
@@
 		(at 199.39 15.24)
 		(size 60.706 28.956)
+		(exclude_from_sim no)
+		(in_bom yes)
+		(on_board yes)
+		(dnp no)
 		(fields_autoplaced yes)
 		(stroke
@@
 		(at 284.226 15.494)
 		(size 40.894 29.718)
+		(exclude_from_sim no)
+		(in_bom yes)
+		(on_board yes)
+		(dnp no)
 		(fields_autoplaced yes)
 		(stroke
@@
 		)
 	)
+	(embedded_fonts no)
 )

Commit message: More cleanup
Parts:
- added H10, H11, H12, H13, H14, H7, H8, H9: MountingHole_Pad, MountingHole:MountingHole_2.2mm_M2_DIN965_Pad, symbol Mechanical:MountingHole_Pad
Connections:
- net GND: now also H10.1, H11.1, H12.1, H13.1, H14.1, H7.1, H8.1, H9.1
