File: hermod-mk2-mx-north/hermod-right/matrix.kicad_sch (KiCad schematic)
At the start: 88 parts

Commit message: Fixed masking issue with PCBs
Parts:
- CH38, CH39: footprint ModHob:KS33_Choc-v2_HS_1U -> ModHob:KS33_Choc-v2_HS_1.5U
- CH41, CH42: footprint ModHob:KS33_Choc-v2_HS_1.5U -> ModHob:KS33_Choc-v2_HS_1U
Changed lines of the file:
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@@
 			)
 		)
-		(property "Footprint" "ModHob:KS33_Choc-v2_HS_1.5U"
+		(property "Footprint" "ModHob:KS33_Choc-v2_HS_1U"
 			(at 194.31 210.82 0)
 			(effects
@@
 			)
 		)
-		(property "Footprint" "ModHob:KS33_Choc-v2_HS_1U"
+		(property "Footprint" "ModHob:KS33_Choc-v2_HS_1.5U"
 			(at 140.97 210.82 0)
 			(effects
@@
 			)
 		)
-		(property "Footprint" "ModHob:KS33_Choc-v2_HS_1U"
+		(property "Footprint" "ModHob:KS33_Choc-v2_HS_1.5U"
 			(at 158.75 210.82 0)
 			(effects
@@
 			)
 		)
-		(property "Footprint" "ModHob:KS33_Choc-v2_HS_1.5U"
+		(property "Footprint" "ModHob:KS33_Choc-v2_HS_1U"
 			(at 212.09 186.69 0)
 			(effects
