File: hermod-mk2-mx/hermod-numpad/numpad.kicad_sch (KiCad schematic)
At the start: 48 parts

Commit message: UPdated Hermod Mk 2 to have ks33 and choc v2 footprints
Parts:
- CH1, CH10, CH11, CH12, CH13, CH14, CH15, CH16, CH17, CH18, CH19, CH2, CH20, CH3, CH4, CH5, CH6, CH7, CH8, CH9: footprint Gateron_KS33_Hotswap:Gateron-KS33-Hotswap-1U -> ModHob:KS33_Choc-v2_HS_1U
Changed lines of the file:
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@@
 			)
 		)
-		(property "Footprint" "Gateron_KS33_Hotswap:Gateron-KS33-Hotswap-1U"
+		(property "Footprint" "ModHob:KS33_Choc-v2_HS_1U"
 			(at 96.52 143.51 0)
 			(effects
@@
 			)
 		)
-		(property "Footprint" "Gateron_KS33_Hotswap:Gateron-KS33-Hotswap-1U"
+		(property "Footprint" "ModHob:KS33_Choc-v2_HS_1U"
 			(at 78.74 143.51 0)
 			(effects
@@
 			)
 		)
-		(property "Footprint" "Gateron_KS33_Hotswap:Gateron-KS33-Hotswap-1U"
+		(property "Footprint" "ModHob:KS33_Choc-v2_HS_1U"
 			(at 78.74 99.06 0)
 			(effects
@@
 			)
 		)
-		(property "Footprint" "Gateron_KS33_Hotswap:Gateron-KS33-Hotswap-1U"
+		(property "Footprint" "ModHob:KS33_Choc-v2_HS_1U"
 			(at 113.03 143.51 0)
 			(effects
@@
 			)
 		)
-		(property "Footprint" "Gateron_KS33_Hotswap:Gateron-KS33-Hotswap-1U"
+		(property "Footprint" "ModHob:KS33_Choc-v2_HS_1U"
 			(at 60.96 99.06 0)
 			(effects
@@
 			)
 		)
-		(property "Footprint" "Gateron_KS33_Hotswap:Gateron-KS33-Hotswap-1U"
+		(property "Footprint" "ModHob:KS33_Choc-v2_HS_1U"
 			(at 60.96 121.92 0)
 			(effects
@@
 			)
 		)
-		(property "Footprint" "Gateron_KS33_Hotswap:Gateron-KS33-Hotswap-1U"
+		(property "Footprint" "ModHob:KS33_Choc-v2_HS_1U"
 			(at 113.03 99.06 0)
 			(effects
@@
 			)
 		)
-		(property "Footprint" "Gateron_KS33_Hotswap:Gateron-KS33-Hotswap-1U"
+		(property "Footprint" "ModHob:KS33_Choc-v2_HS_1U"
 			(at 96.52 55.88 0)
 			(effects
@@
 			)
 		)
-		(property "Footprint" "Gateron_KS33_Hotswap:Gateron-KS33-Hotswap-1U"
+		(property "Footprint" "ModHob:KS33_Choc-v2_HS_1U"
 			(at 60.96 55.88 0)
 			(effects
@@
 			)
 		)
-		(property "Footprint" "Gateron_KS33_Hotswap:Gateron-KS33-Hotswap-1U"
+		(property "Footprint" "ModHob:KS33_Choc-v2_HS_1U"
 			(at 113.03 55.88 0)
 			(effects
@@
 			)
 		)
-		(property "Footprint" "Gateron_KS33_Hotswap:Gateron-KS33-Hotswap-1U"
+		(property "Footprint" "ModHob:KS33_Choc-v2_HS_1U"
 			(at 78.74 77.47 0)
 			(effects
@@
 			)
 		)
-		(property "Footprint" "Gateron_KS33_Hotswap:Gateron-KS33-Hotswap-1U"
+		(property "Footprint" "ModHob:KS33_Choc-v2_HS_1U"
 			(at 113.03 77.47 0)
 			(effects
@@
 			)
 		)
-		(property "Footprint" "Gateron_KS33_Hotswap:Gateron-KS33-Hotswap-1U"
+		(property "Footprint" "ModHob:KS33_Choc-v2_HS_1U"
 			(at 96.52 77.47 0)
 			(effects
@@
 			)
 		)
-		(property "Footprint" "Gateron_KS33_Hotswap:Gateron-KS33-Hotswap-1U"
+		(property "Footprint" "ModHob:KS33_Choc-v2_HS_1U"
 			(at 96.52 99.06 0)
 			(effects
@@
 			)
 		)
-		(property "Footprint" "Gateron_KS33_Hotswap:Gateron-KS33-Hotswap-1U"
+		(property "Footprint" "ModHob:KS33_Choc-v2_HS_1U"
 			(at 113.03 121.92 0)
 			(effects
@@
 			)
 		)
-		(property "Footprint" "Gateron_KS33_Hotswap:Gateron-KS33-Hotswap-1U"
+		(property "Footprint" "ModHob:KS33_Choc-v2_HS_1U"
 			(at 60.96 143.51 0)
 			(effects
@@
 			)
 		)
-		(property "Footprint" "Gateron_KS33_Hotswap:Gateron-KS33-Hotswap-1U"
+		(property "Footprint" "ModHob:KS33_Choc-v2_HS_1U"
 			(at 78.74 55.88 0)
 			(effects
@@
 			)
 		)
-		(property "Footprint" "Gateron_KS33_Hotswap:Gateron-KS33-Hotswap-1U"
+		(property "Footprint" "ModHob:KS33_Choc-v2_HS_1U"
 			(at 78.74 121.92 0)
 			(effects
@@
 			)
 		)
-		(property "Footprint" "Gateron_KS33_Hotswap:Gateron-KS33-Hotswap-1U"
+		(property "Footprint" "ModHob:KS33_Choc-v2_HS_1U"
 			(at 96.52 121.92 0)
 			(effects
@@
 			)
 		)
-		(property "Footprint" "Gateron_KS33_Hotswap:Gateron-KS33-Hotswap-1U"
+		(property "Footprint" "ModHob:KS33_Choc-v2_HS_1U"
 			(at 60.96 77.47 0)
 			(effects
